Commit message: feat: add robotiq_2f-85 gripper description and moveit group

File: src/arm_description/urdf/ur.ros2_control.xacro (robot description, xacro)
@@ -45,4 +45,47 @@
       <xacro:arm_joint_interface joint_name="wrist_2_joint" initial_value="${initial_positions['wrist_2_joint']}"/>
       <xacro:arm_joint_interface joint_name="wrist_3_joint" initial_value="${initial_positions['wrist_3_joint']}"/>
+      <joint name="robotiq_85_left_knuckle_joint">
+        <command_interface name="position">
+          <param name="min">0.0</param>
+          <param name="max">0.8</param>
+        </command_interface>
+        <state_interface name="position"/>
+        <state_interface name="velocity"/>
+      </joint>
+      <joint name="robotiq_85_right_knuckle_joint">
+        <param name="mimic">robotiq_85_left_knuckle_joint</param>
+        <param name="multiplier">-1</param>
+        <command_interface name="position"/>
+        <state_interface name="position"/>
+        <state_interface name="velocity"/>
+      </joint>
+      <joint name="robotiq_85_left_inner_knuckle_joint">
+        <param name="mimic">robotiq_85_left_knuckle_joint</param>
+        <param name="multiplier">1</param>
+        <command_interface name="position"/>
+        <state_interface name="position"/>
+        <state_interface name="velocity"/>
+      </joint>
+      <joint name="robotiq_85_right_inner_knuckle_joint">
+        <param name="mimic">robotiq_85_left_knuckle_joint</param>
+        <param name="multiplier">-1</param>
+        <command_interface name="position"/>
+        <state_interface name="position"/>
+        <state_interface name="velocity"/>
+      </joint>
+      <joint name="robotiq_85_left_finger_tip_joint">
+        <param name="mimic">robotiq_85_left_knuckle_joint</param>
+        <param name="multiplier">-1</param>
+        <command_interface name="position"/>
+        <state_interface name="position"/>
+        <state_interface name="velocity"/>
+      </joint>
+      <joint name="robotiq_85_right_finger_tip_joint">
+        <param name="mimic">robotiq_85_left_knuckle_joint</param>
+        <param name="multiplier">1</param>
+        <command_interface name="position"/>
+        <state_interface name="position"/>
+        <state_interface name="velocity"/>
+      </joint>
     </ros2_control>
   </xacro:macro>

File: src/arm_description/urdf/ur.urdf.xacro (robot description, xacro)
@@ -5,4 +5,6 @@
    <!-- import main macro -->
    <xacro:include filename="$(find arm_description)/urdf/ur_macro.xacro"/>
+   <xacro:include filename="$(find robotiq_description)/urdf/ur_to_robotiq_adapter.urdf.xacro"/>
+   <xacro:include filename="$(find robotiq_description)/urdf/robotiq_2f_85_macro.urdf.xacro"/>
    <!-- parameters -->
    <xacro:arg name="tf_prefix" default="" />
@@ -72,4 +74,18 @@
      <origin xyz="0 0 0" rpy="0 0 0" />          <!-- position robot in the world -->
    </xacro:ur_robot>
+   <xacro:ur_to_robotiq prefix="" parent="tool0" child="robotiq_85_mount_link"/>
+   <xacro:robotiq_gripper
+     name="robotiq_85"
+     prefix=""
+     parent="robotiq_85_mount_link"
+     include_ros2_control="false">
+     <origin xyz="0 0 0" rpy="0 0 0"/>
+   </xacro:robotiq_gripper>
+   <link name="tcp"/>
+   <joint name="tcp_joint" type="fixed">
+     <parent link="robotiq_85_base_link"/>
+     <child link="tcp"/>
+     <origin xyz="0 0 0.16" rpy="0 0 0"/>
+   </joint>
    <xacro:if value="$(arg sim_gazebo)">
     <!-- Gazebo plugins -->

File: src/arm_moveit_config/srdf/arm_macro.srdf.xacro (robot description, xacro)
@@ -12,5 +12,8 @@
     <!--SUBGROUPS - Groups can also be formed by referencing to already defined group names-->
     <group name="${prefix}${name}_manipulator">
-      <chain base_link="${prefix}base_link" tip_link="${prefix}tool0" />
+      <chain base_link="${prefix}base_link" tip_link="${prefix}tcp" />
+    </group>
+    <group name="${prefix}gripper">
+      <joint name="${prefix}robotiq_85_left_knuckle_joint" />
     </group>
     <!--GROUP STATES - Purpose - Define a named state for a particular group, in terms of joint values. This is useful to define states like 'folded arms'-->
@@ -39,5 +42,12 @@
       <joint name="${prefix}wrist_3_joint" value="-0.11" />
     </group_state>
+    <group_state name="${prefix}open" group="${prefix}gripper">
+      <joint name="${prefix}robotiq_85_left_knuckle_joint" value="0.0" />
+    </group_state>
+    <group_state name="${prefix}closed" group="${prefix}gripper">
+      <joint name="${prefix}robotiq_85_left_knuckle_joint" value="0.8" />
+    </group_state>
     <!--END EFFECTOR - Purpose - Represent information about an end effector.-->
+    <end_effector name="${prefix}gripper" parent_link="${prefix}tool0" group="${prefix}gripper" parent_group="${prefix}${name}_manipulator" />
     <!--VIRTUAL JOINT - Purpose - this element defines a virtual joint between a robot link and an external frame of reference (considered fixed with respect to the robot)-->
     <!--DISABLE COLLISIONS - By default it is assumed that any link of the robot could potentially come into collision with any other link in the robot. This tag disables collision checking between a specified pair of links. -->
@@ -53,4 +63,33 @@
     <disable_collisions link1="${prefix}wrist_1_link" link2="${prefix}wrist_3_link" reason="Never" />
     <disable_collisions link1="${prefix}wrist_2_link" link2="${prefix}wrist_3_link" reason="Adjacent" />
+    <disable_collisions link1="${prefix}flange" link2="${prefix}tool0" reason="Adjacent" />
+    <disable_collisions link1="${prefix}flange" link2="${prefix}ur_to_robotiq_link" reason="Never" />
+    <disable_collisions link1="${prefix}flange" link2="${prefix}robotiq_85_mount_link" reason="Never" />
+    <disable_collisions link1="${prefix}flange" link2="${prefix}robotiq_85_base_link" reason="Never" />
+    <disable_collisions link1="${prefix}tool0" link2="${prefix}ur_to_robotiq_link" reason="Adjacent" />
+    <disable_collisions link1="${prefix}tool0" link2="${prefix}robotiq_85_base_link" reason="Never" />
+    <disable_collisions link1="${prefix}wrist_3_link" link2="${prefix}ur_to_robotiq_link" reason="Never" />
+    <disable_collisions link1="${prefix}wrist_3_link" link2="${prefix}robotiq_85_base_link" reason="Never" />
+    <disable_collisions link1="${prefix}ur_to_robotiq_link" link2="${prefix}robotiq_85_mount_link" reason="Adjacent" />
+    <disable_collisions link1="${prefix}ur_to_robotiq_link" link2="${prefix}robotiq_85_base_link" reason="Never" />
+    <disable_collisions link1="${prefix}robotiq_85_mount_link" link2="${prefix}robotiq_85_base_link" reason="Adjacent" />
+    <disable_collisions link1="${prefix}robotiq_85_base_link" link2="${prefix}robotiq_85_left_knuckle_link" reason="Adjacent" />
+    <disable_collisions link1="${prefix}robotiq_85_base_link" link2="${prefix}robotiq_85_right_knuckle_link" reason="Adjacent" />
+    <disable_collisions link1="${prefix}robotiq_85_base_link" link2="${prefix}robotiq_85_left_inner_knuckle_link" reason="Adjacent" />
+    <disable_collisions link1="${prefix}robotiq_85_base_link" link2="${prefix}robotiq_85_right_inner_knuckle_link" reason="Adjacent" />
+    <disable_collisions link1="${prefix}robotiq_85_left_knuckle_link" link2="${prefix}robotiq_85_left_finger_link" reason="Adjacent" />
+    <disable_collisions link1="${prefix}robotiq_85_right_knuckle_link" link2="${prefix}robotiq_85_right_finger_link" reason="Adjacent" />
+    <disable_collisions link1="${prefix}robotiq_85_left_finger_link" link2="${prefix}robotiq_85_left_finger_tip_link" reason="Adjacent" />
+    <disable_collisions link1="${prefix}robotiq_85_right_finger_link" link2="${prefix}robotiq_85_right_finger_tip_link" reason="Adjacent" />
+    <disable_collisions link1="${prefix}robotiq_85_left_knuckle_link" link2="${prefix}robotiq_85_left_inner_knuckle_link" reason="Never" />
+    <disable_collisions link1="${prefix}robotiq_85_right_knuckle_link" link2="${prefix}robotiq_85_right_inner_knuckle_link" reason="Never" />
+    <disable_collisions link1="${prefix}robotiq_85_left_finger_link" link2="${prefix}robotiq_85_left_inner_knuckle_link" reason="Never" />
+    <disable_collisions link1="${prefix}robotiq_85_right_finger_link" link2="${prefix}robotiq_85_right_inner_knuckle_link" reason="Never" />
+    <disable_collisions link1="${prefix}robotiq_85_left_finger_tip_link" link2="${prefix}robotiq_85_left_inner_knuckle_link" reason="Never" />
+    <disable_collisions link1="${prefix}robotiq_85_right_finger_tip_link" link2="${prefix}robotiq_85_right_inner_knuckle_link" reason="Never" />
+    <disable_collisions link1="${prefix}robotiq_85_left_finger_tip_link" link2="${prefix}robotiq_85_right_finger_tip_link" reason="Never" />
+    <disable_collisions link1="${prefix}robotiq_85_left_finger_link" link2="${prefix}robotiq_85_right_finger_link" reason="Never" />
+    <disable_collisions link1="${prefix}robotiq_85_left_inner_knuckle_link" link2="${prefix}robotiq_85_right_inner_knuckle_link" reason="Never" />
+    <disable_collisions link1="${prefix}robotiq_85_left_knuckle_link" link2="${prefix}robotiq_85_right_knuckle_link" reason="Never" />
   </xacro:macro>
 </robot>
