Commit message: feat: add pick_place_static logic

File: src/arm_description/urdf/ur.urdf.xacro (robot description, xacro)
@@ -16,4 +16,5 @@
    <xacro:arg name="safety_pos_margin" default="0.15"/>
    <xacro:arg name="safety_k_position" default="20"/>
+   <xacro:arg name="robot_base_z" default="0.0"/>
      <!-- Simulation parameters -->
    <xacro:arg name="use_fake_hardware" default="false" />
@@ -72,5 +73,5 @@
      initial_positions="${xacro.load_yaml(initial_positions_file)}"
      >
-     <origin xyz="0 0 0" rpy="0 0 0" />          <!-- position robot in the world -->
+     <origin xyz="0 0 $(arg robot_base_z)" rpy="0 0 0" />          <!-- position robot in the world -->
    </xacro:ur_robot>
    <xacro:ur_to_robotiq prefix="" parent="tool0" child="robotiq_85_mount_link"/>

Commit message: feat: add pick_place_dynamic logic

File: src/arm_description/urdf/ur.urdf.xacro (robot description, xacro)
@@ -83,4 +83,60 @@
      <origin xyz="0 0 0" rpy="0 0 0"/>
    </xacro:robotiq_gripper>
+   <link name="wrist_camera_link">
+     <visual>
+       <origin xyz="0 0 0" rpy="0 0 0"/>
+       <geometry>
+         <box size="0.035 0.025 0.025"/>
+       </geometry>
+       <material name="wrist_camera_black">
+         <color rgba="0.02 0.02 0.02 1.0"/>
+       </material>
+     </visual>
+     <collision>
+       <origin xyz="0 0 0" rpy="0 0 0"/>
+       <geometry>
+         <box size="0.035 0.025 0.025"/>
+       </geometry>
+     </collision>
+     <inertial>
+       <origin xyz="0 0 0" rpy="0 0 0"/>
+       <mass value="0.02"/>
+       <inertia ixx="0.000001" ixy="0" ixz="0" iyy="0.000001" iyz="0" izz="0.000001"/>
+     </inertial>
+   </link>
+   <joint name="wrist_camera_joint" type="fixed">
+     <parent link="tool0"/>
+     <child link="wrist_camera_link"/>
+     <origin xyz="0 -0.06 0.03" rpy="0 -1.5708 0"/>
+   </joint>
+   <link name="wrist_camera_optical_frame"/>
+   <joint name="wrist_camera_optical_joint" type="fixed">
+     <parent link="wrist_camera_link"/>
+     <child link="wrist_camera_optical_frame"/>
+     <origin xyz="0 0 0" rpy="-1.5708 0 -1.5708"/>
+   </joint>
+   <xacro:if value="$(arg sim_ignition)">
+     <gazebo reference="wrist_camera_link">
+       <sensor name="wrist_camera" type="rgbd_camera">
+         <pose>0 0 0 0 0 0</pose>
+         <always_on>true</always_on>
+         <update_rate>15</update_rate>
+         <topic>wrist_camera</topic>
+         <gz_frame_id>wrist_camera_optical_frame</gz_frame_id>
+         <camera>
+           <horizontal_fov>1.21</horizontal_fov>
+           <image>
+             <width>640</width>
+             <height>480</height>
+             <format>R8G8B8</format>
+           </image>
+           <clip>
+             <near>0.2</near>
+             <far>3.0</far>
+           </clip>
+         </camera>
+       </sensor>
+     </gazebo>
+   </xacro:if>
    <link name="tcp"/>
    <joint name="tcp_joint" type="fixed">
